File: multitool_two_v1.kicad_sch (KiCad schematic)
At the start: 69 parts, among them J1 Conn_02x08_Odd_Even, SW1 SW_Push, SW2 SW_Push, SW3 SW_Push, SW4 SW_Push, SW5 SW_Push, SW6 SW_Push, SW7 SW_Push, SW8 SW_Push, U1 4017, U2 74LS74, U3 74LS74, U4 74LS74, U5 74LS74, U6 74HCT00, U7 74HCT00, U8 74HCT00

Commit message: committing with a bug
Parts:
- removed unit 5 of U6
- removed unit 5 of U7
- removed unit 5 of U8
- added C10, C11, C12, C13, C14, C15, C16, C17, C18, C19, C20, C21, C22, C23, C24, C25, C26, C27, C28, C29, C30, C31, C32, C33, C34, C35, C36, C37, C38, C39, C40, C41, C42, C43, C44, C45, C46, C47, C48, C49, C50, C51, C52, C53, C54, C55, C56, C57, C58, C59, C60, C61, C62, C63, C64, C9: 1u, Capacitor_SMD:C_0603_1608Metric, symbol Device:C
- added D10, D11, D12, D13, D14, D15, D16, D17, D18, D19, D20, D21, D22, D23, D24, D25, D26, D27, D28, D29, D30, D31, D32, D33, D34, D35, D36, D37, D38, D39, D40, D41, D42, D43, D44, D45, D46, D47, D48, D49, D50, D51, D52, D53, D54, D55, D56, D57, D58, D59, D60, D61, D62, D63, D64, D9: DIODE, Diode_SMD:D_SOD-323F, symbol pspice:DIODE
- added DL1, DL18, DL19, DL2, DL20, DL21, DL22, DL23, DL24, DL25, DL26, DL27, DL28, DL29, DL3, DL30, DL31, DL32, DL33, DL34, DL35, DL36, DL37, DL38, DL39, DL4, DL40, DL41, DL42, DL43, DL44, DL45, DL46, DL47, DL48, DL49, DL5, DL50, DL51, DL52, DL53, DL54, DL55, DL56, DL57, DL58, DL59, DL6, DL60, DL61, DL62, DL63, DL64, DL65, DL66, DL67, DL68, DL69, DL7, DL70, DL71, DL72, DL8: LED, LED_SMD:LED_0603_1608Metric, symbol Device:LED
- added JOUT2, JOUT3, JOUT4, JOUT5, JOUT6, JOUT7, JOUT8: AudioJack2_SwitchT, Connector_Audio:Jack_3.5mm_QingPu_WQP-PJ398SM_Vertical_CircularHoles, symbol Connector:AudioJack2_SwitchT
- added R100, R101, R102, R103, R104, R105, R106, R107, R108, R109, R110, R111, R112, R113, R114, R115, R116, R133, R134, R135, R136, R137, R138, R139, R140, R141, R142, R143, R144, R145, R146, R147, R148, R149, R150, R151, R152, R153, R154, R155, R156, R157, R158, R159, R160, R161, R162, R163, R164, R165, R166, R183, R184, R185, R186, R187, R188, R189, R190, R191, R192, R193, R194, R195, R196, R197, R198, R199, R200, R26, R27, R28, R29, R30, R31, R32, R33, R42, R43, R44, R45, R46, R47, R48, R49, R50, R51, R52, R53, R54, R55, R56, R57, R58, R59, R60, R61, R62, R63, R64, R65, R66, R83, R84, R85, R86, R87, R88, R89, R90, R91, R92, R93, R94, R95, R96, R97, R98, R99: 1k, Resistor_SMD:R_0603_1608Metric, symbol Device:R
- added R117, R118, R119, R120, R121, R122, R123, R124, R125, R126, R127, R128, R129, R130, R131, R132, R167, R168, R169, R170, R171, R172, R173, R174, R175, R176, R177, R178, R179, R180, R181, R182, R34, R35, R36, R37, R38, R39, R40, R41, R67, R68, R69, R70, R71, R72, R73, R74, R75, R76, R77, R78, R79, R80, R81, R82: 10k, Resistor_SMD:R_0603_1608Metric, symbol Device:R
- added SW10, SW11, SW12, SW13, SW14, SW15, SW16, SW17, SW18, SW19, SW20, SW21, SW22, SW23, SW24, SW25, SW26, SW27, SW28, SW29, SW30, SW31, SW32, SW33, SW34, SW35, SW36, SW37, SW38, SW39, SW40, SW41, SW42, SW43, SW44, SW45, SW46, SW47, SW48, SW49, SW50, SW51, SW52, SW53, SW54, SW55, SW56, SW57, SW58, SW59, SW60, SW61, SW62, SW63, SW64, SW9: SW_Push, Button_Switch_SMD:SW_SPST_B3S-1000, symbol Switch:SW_Push
- added unit 5 of UAND_1
- added UAND_10, UAND_11, UAND_12, UAND_13, UAND_14, UAND_15, UAND_16, UAND_18, UAND_3, UAND_4, UAND_5, UAND_6, UAND_7, UAND_8, UAND_9: 74HCT00, Package_SO:SO-14_3.9x8.65mm_P1.27mm, symbol 74xx:74HCT00
- added unit 5 of UAND_17
- added unit 5 of UAND_2
- added UFLIP_10, UFLIP_11, UFLIP_12, UFLIP_13, UFLIP_14, UFLIP_15, UFLIP_16, UFLIP_17, UFLIP_18, UFLIP_19, UFLIP_20, UFLIP_21, UFLIP_22, UFLIP_23, UFLIP_24, UFLIP_25, UFLIP_26, UFLIP_27, UFLIP_28, UFLIP_29, UFLIP_30, UFLIP_31, UFLIP_32, UFLIP_5, UFLIP_6, UFLIP_7, UFLIP_8, UFLIP_9: 74LS74, Package_SO:SOIC-14_3.9x8.7mm_P1.27mm, symbol 74xx:74LS74
- renumbered U6 to UAND_1, U8 to UAND_17, U7 to UAND_2, U2 to UFLIP_1, U3 to UFLIP_2, U4 to UFLIP_3, U5 to UFLIP_4
Connections:
- net +5V: now also SW10.1, SW11.1, SW12.1, SW13.1, SW14.1, SW15.1, SW16.1, SW17.1, SW18.1, SW19.1, SW20.1, SW21.1, SW22.1, SW23.1, SW24.1, SW25.1, SW26.1, SW27.1, SW28.1, SW29.1, SW30.1, SW31.1, SW32.1, SW33.1, SW34.1, SW35.1, SW36.1, SW37.1, SW38.1, SW39.1, SW40.1, SW41.1, SW42.1, SW43.1, SW44.1, SW45.1, SW46.1, SW47.1, SW48.1, SW49.1, SW50.1, SW51.1, SW52.1, SW53.1, SW54.1, SW55.1, SW56.1, SW57.1, SW58.1, SW59.1, SW60.1, SW61.1, SW62.1, SW63.1, SW64.1, SW9.1, UAND_1.14 (VCC), UAND_10.14 (VCC), UAND_11.14 (VCC), UAND_12.14 (VCC), UAND_13.14 (VCC), UAND_14.14 (VCC), UAND_15.14 (VCC), UAND_16.14 (VCC), UAND_17.14 (VCC), UAND_18.14 (VCC), UAND_2.14 (VCC), UAND_3.14 (VCC), UAND_4.14 (VCC), UAND_5.14 (VCC), UAND_6.14 (VCC), UAND_7.14 (VCC), UAND_8.14 (VCC), UAND_9.14 (VCC), UFLIP_10.10 (~S), UFLIP_10.14 (VCC), UFLIP_10.4 (~S), UFLIP_11.10 (~S), UFLIP_11.14 (VCC), UFLIP_11.4 (~S), UFLIP_12.10 (~S), UFLIP_12.14 (VCC), UFLIP_12.4 (~S), UFLIP_13.10 (~S), UFLIP_13.14 (VCC), UFLIP_13.4 (~S), UFLIP_14.10 (~S), UFLIP_14.14 (VCC), UFLIP_14.4 (~S), UFLIP_15.10 (~S), UFLIP_15.14 (VCC), UFLIP_15.4 (~S), UFLIP_16.10 (~S), UFLIP_16.14 (VCC), UFLIP_16.4 (~S), UFLIP_17.10 (~S), UFLIP_17.14 (VCC), UFLIP_17.4 (~S), UFLIP_18.10 (~S), UFLIP_18.14 (VCC), UFLIP_18.4 (~S), UFLIP_19.10 (~S), UFLIP_19.14 (VCC), UFLIP_19.4 (~S), UFLIP_20.10 (~S), UFLIP_20.14 (VCC), UFLIP_20.4 (~S), UFLIP_21.10 (~S), UFLIP_21.14 (VCC), UFLIP_21.4 (~S), UFLIP_22.10 (~S), UFLIP_22.14 (VCC), UFLIP_22.4 (~S), UFLIP_23.10 (~S), UFLIP_23.14 (VCC), UFLIP_23.4 (~S), UFLIP_24.10 (~S), UFLIP_24.14 (VCC), UFLIP_24.4 (~S), UFLIP_25.10 (~S), UFLIP_25.14 (VCC), UFLIP_25.4 (~S), UFLIP_26.10 (~S), UFLIP_26.14 (VCC), UFLIP_26.4 (~S), UFLIP_27.10 (~S), UFLIP_27.14 (VCC), UFLIP_27.4 (~S), UFLIP_28.10 (~S), UFLIP_28.14 (VCC), UFLIP_28.4 (~S), UFLIP_29.10 (~S), UFLIP_29.14 (VCC), UFLIP_29.4 (~S), UFLIP_30.10 (~S), UFLIP_30.14 (VCC), UFLIP_30.4 (~S), UFLIP_31.10 (~S), UFLIP_31.14 (VCC), UFLIP_31.4 (~S), UFLIP_32.10 (~S), UFLIP_32.14 (VCC), UFLIP_32.4 (~S), UFLIP_5.10 (~S), UFLIP_5.14 (VCC), UFLIP_5.4 (~S), UFLIP_6.10 (~S), UFLIP_6.14 (VCC), UFLIP_6.4 (~S), UFLIP_7.10 (~S), UFLIP_7.14 (VCC), UFLIP_7.4 (~S), UFLIP_8.10 (~S), UFLIP_8.14 (VCC), UFLIP_8.4 (~S), UFLIP_9.10 (~S), UFLIP_9.14 (VCC), UFLIP_9.4 (~S)
- net GND: now also C10.2, C11.2, C12.2, C13.2, C14.2, C15.2, C16.2, C17.2, C18.2, C19.2, C20.2, C21.2, C22.2, C23.2, C24.2, C25.2, C26.2, C27.2, C28.2, C29.2, C30.2, C31.2, C32.2, C33.2, C34.2, C35.2, C36.2, C37.2, C38.2, C39.2, C40.2, C41.2, C42.2, C43.2, C44.2, C45.2, C46.2, C47.2, C48.2, C49.2, C50.2, C51.2, C52.2, C53.2, C54.2, C55.2, C56.2, C57.2, C58.2, C59.2, C60.2, C61.2, C62.2, C63.2, C64.2, C9.2, JOUT2.S, JOUT3.S, JOUT4.S, JOUT5.S, JOUT6.S, JOUT7.S, JOUT8.S, R100.2, R117.1, R118.1, R119.1, R120.1, R121.1, R122.1, R123.1, R124.1, R125.1, R126.1, R127.1, R128.1, R129.1, R130.1, R131.1, R132.1, R133.2, R134.2, R135.2, R136.2, R137.2, R138.2, R139.2, R140.2, R141.2, R142.2, R143.2, R144.2, R145.2, R146.2, R147.2, R148.2, R149.2, R150.2, R167.1, R168.1, R169.1, R170.1, R171.1, R172.1, R173.1, R174.1, R175.1, R176.1, R177.1, R178.1, R179.1, R180.1, R181.1, R182.1, R183.2, R184.2, R185.2, R186.2, R187.2, R188.2, R189.2, R190.2, R191.2, R192.2, R193.2, R194.2, R195.2, R196.2, R197.2, R198.2, R199.2, R200.2, R34.1, R35.1, R36.1, R37.1, R38.1, R39.1, R40.1, R41.1, R42.2, R43.2, R44.2, R45.2, R46.2, R47.2, R48.2, R49.2, R50.2, R67.1, R68.1, R69.1, R70.1, R71.1, R72.1, R73.1, R74.1, R75.1, R76.1, R77.1, R78.1, R79.1, R80.1, R81.1, R82.1, R83.2, R84.2, R85.2, R86.2, R87.2, R88.2, R89.2, R90.2, R91.2, R92.2, R93.2, R94.2, R95.2, R96.2, R97.2, R98.2, R99.2, UAND_1.7 (GND), UAND_10.7 (GND), UAND_11.7 (GND), UAND_12.7 (GND), UAND_13.7 (GND), UAND_14.7 (GND), UAND_15.7 (GND), UAND_16.7 (GND), UAND_17.7 (GND), UAND_18.7 (GND), UAND_2.7 (GND), UAND_3.7 (GND), UAND_4.7 (GND), UAND_5.7 (GND), UAND_6.7 (GND), UAND_7.7 (GND), UAND_8.7 (GND), UAND_9.7 (GND), UFLIP_10.1 (~R), UFLIP_10.13 (~R), UFLIP_10.7 (GND), UFLIP_11.1 (~R), UFLIP_11.13 (~R), UFLIP_11.7 (GND), UFLIP_12.1 (~R), UFLIP_12.13 (~R), UFLIP_12.7 (GND), UFLIP_13.1 (~R), UFLIP_13.13 (~R), UFLIP_13.7 (GND), UFLIP_14.1 (~R), UFLIP_14.13 (~R), UFLIP_14.7 (GND), UFLIP_15.1 (~R), UFLIP_15.13 (~R), UFLIP_15.7 (GND), UFLIP_16.1 (~R), UFLIP_16.13 (~R), UFLIP_16.7 (GND), UFLIP_17.1 (~R), UFLIP_17.13 (~R), UFLIP_17.7 (GND), UFLIP_18.1 (~R), UFLIP_18.13 (~R), UFLIP_18.7 (GND), UFLIP_19.1 (~R), UFLIP_19.13 (~R), UFLIP_19.7 (GND), UFLIP_20.1 (~R), UFLIP_20.13 (~R), UFLIP_20.7 (GND), UFLIP_21.1 (~R), UFLIP_21.13 (~R), UFLIP_21.7 (GND), UFLIP_22.1 (~R), UFLIP_22.13 (~R), UFLIP_22.7 (GND), UFLIP_23.1 (~R), UFLIP_23.13 (~R), UFLIP_23.7 (GND), UFLIP_24.1 (~R), UFLIP_24.13 (~R), UFLIP_24.7 (GND), UFLIP_25.1 (~R), UFLIP_25.13 (~R), UFLIP_25.7 (GND), UFLIP_26.1 (~R), UFLIP_26.13 (~R), UFLIP_26.7 (GND), UFLIP_27.1 (~R), UFLIP_27.13 (~R), UFLIP_27.7 (GND), UFLIP_28.1 (~R), UFLIP_28.13 (~R), UFLIP_28.7 (GND), UFLIP_29.1 (~R), UFLIP_29.13 (~R), UFLIP_29.7 (GND), UFLIP_30.1 (~R), UFLIP_30.13 (~R), UFLIP_30.7 (GND), UFLIP_31.1 (~R), UFLIP_31.13 (~R), UFLIP_31.7 (GND), UFLIP_32.1 (~R), UFLIP_32.13 (~R), UFLIP_32.7 (GND), UFLIP_5.1 (~R), UFLIP_5.13 (~R), UFLIP_5.7 (GND), UFLIP_6.1 (~R), UFLIP_6.13 (~R), UFLIP_6.7 (GND), UFLIP_7.1 (~R), UFLIP_7.13 (~R), UFLIP_7.7 (GND), UFLIP_8.1 (~R), UFLIP_8.13 (~R), UFLIP_8.7 (GND), UFLIP_9.1 (~R), UFLIP_9.13 (~R), UFLIP_9.7 (GND)
- net clock: now also UAND_17.10, UAND_17.13, UAND_17.5, UAND_18.10, UAND_18.13, UAND_18.2, UAND_18.5
- net count_1: now also UAND_11.1, UAND_13.1, UAND_15.1, UAND_3.1, UAND_5.1, UAND_7.1, UAND_9.1
- net count_2: now also UAND_11.4, UAND_13.4, UAND_15.4, UAND_3.4, UAND_5.4, UAND_7.4, UAND_9.4
- net count_3: now also UAND_11.9, UAND_13.9, UAND_15.9, UAND_3.9, UAND_5.9, UAND_7.9, UAND_9.9
- net count_4: now also UAND_11.12, UAND_13.12, UAND_15.12, UAND_3.12, UAND_5.12, UAND_7.12, UAND_9.12
- net count_5: now also UAND_10.1, UAND_12.1, UAND_14.1, UAND_16.1, UAND_4.1, UAND_6.1, UAND_8.1
- net count_6: now also UAND_10.4, UAND_12.4, UAND_14.4, UAND_16.4, UAND_4.4, UAND_6.4, UAND_8.4
- net count_7: now also UAND_10.9, UAND_12.9, UAND_14.9, UAND_16.9, UAND_4.9, UAND_6.9, UAND_8.9
- net count_8: now also UAND_10.12, UAND_12.12, UAND_14.12, UAND_16.12, UAND_4.12, UAND_6.12, UAND_8.12
- net at UAND_17.8: now also DL54.2 (A), JOUT6.T
- net at UAND_17.9: now also D41.2 (A), D42.2 (A), D43.2 (A), D44.2 (A), D45.2 (A), D46.2 (A), D47.2 (A), D48.2 (A)
- net at UAND_17.4: now also D25.2 (A), D26.2 (A), D27.2 (A), D28.2 (A), D29.2 (A), D30.2 (A), D31.2 (A), D32.2 (A)
- net at UAND_17.6: now also DL36.2 (A), JOUT4.T
- net at UAND_17.11: now also DL72.2 (A), JOUT8.T
- net at UAND_17.12: now also D57.2 (A), D58.2 (A), D59.2 (A), D60.2 (A), D61.2 (A), D62.2 (A), D63.2 (A), D64.2 (A)
- new net: R106.1, SW38.2
- new net: C44.1, R112.2, R128.2, UFLIP_10.11 (C)
- new net: DL2.1 (K), R43.1
- new net: D38.1 (K), UAND_14.6
- new net: D33.2 (A), D34.2 (A), D35.2 (A), D36.2 (A), D37.2 (A), D38.2 (A), D39.2 (A), D40.2 (A), UAND_18.9
- new net: D63.1 (K), UAND_8.8
- new net: DL2.2 (A), UAND_9.5, UFLIP_17.9 (Q)
- new net: C22.1, R56.2, R72.2, UFLIP_23.11 (C)
- new net: UFLIP_23.12 (D), UFLIP_23.8 (~Q)
- new net: DL24.2 (A), UAND_12.5, UFLIP_23.9 (Q)
- new net: D60.1 (K), UAND_7.11
- new net: DL66.2 (A), UAND_7.13, UFLIP_14.9 (Q)
- new net: C32.1, R66.2, R82.2, UFLIP_8.11 (C)
- new net: UFLIP_8.12 (D), UFLIP_8.8 (~Q)
- new net: DL34.2 (A), UAND_4.13, UFLIP_8.9 (Q)
- new net: DL18.1 (K), R50.1
- new net: R108.1, SW40.2
- new net: R110.1, SW42.2
- new net: C42.1, R110.2, R126.2, UFLIP_9.11 (C)
- new net: C50.1, R152.2, R168.2, UFLIP_29.11 (C)
- new net: DL47.1 (K), R143.1
- new net: DL47.2 (A), UAND_5.10, UFLIP_10.5 (Q)
- new net: R66.1, SW32.2
- new net: C14.1, R31.2, R39.2, UFLIP_19.11 (C)
- new net: UFLIP_19.12 (D), UFLIP_19.8 (~Q)
- new net: DL6.2 (A), UAND_10.5, UFLIP_19.9 (Q)
- new net: DL69.1 (K), R197.1
- new net: DL69.2 (A), UAND_8.10, UFLIP_16.5 (Q)
- new net: DL46.1 (K), R142.1
- new net: DL46.2 (A), UAND_5.5, UFLIP_9.9 (Q)
- new net: DL55.1 (K), R183.1
- new net: R103.1, SW35.2
- new net: C52.1, R154.2, R170.2, UFLIP_30.11 (C)
- new net: UFLIP_30.12 (D), UFLIP_30.8 (~Q)
- new net: DL58.2 (A), UAND_15.13, UFLIP_30.9 (Q)
- new net: D58.1 (K), UAND_7.6
- new net: R52.1, SW18.2
- new net: C18.1, R52.2, R68.2, UFLIP_21.11 (C)
- new net: DL52.1 (K), R148.1
- new net: C27.1, R61.2, R77.2, UFLIP_6.3 (C)
- new net: DL42.1 (K), R138.1
- new net: DL42.2 (A), UAND_14.5, UFLIP_27.9 (Q)
- new net: DL65.2 (A), UAND_7.10, UFLIP_14.5 (Q)
- new net: D59.1 (K), UAND_7.8
- new net: D64.1 (K), UAND_8.11
- new net: DL70.2 (A), UAND_8.13, UFLIP_16.9 (Q)
- new net: DL53.1 (K), R149.1
- new net: DL39.1 (K), R135.1
- new net: DL39.2 (A), UAND_13.10, UFLIP_26.5 (Q)
- new net: C25.1, R59.2, R75.2, UFLIP_5.3 (C)
- new net: C28.1, R62.2, R78.2, UFLIP_6.11 (C)
- new net: C9.1, R26.2, R34.2, UFLIP_17.3 (C)
- new net: DL45.1 (K), R141.1
- new net: DL68.1 (K), R196.1
- new net: D44.1 (K), UAND_5.11
- new net: DL48.2 (A), UAND_5.13, UFLIP_10.9 (Q)
- new net: R113.1, SW45.2
- new net: R27.1, SW10.2
- new net: DL8.1 (K), R49.1
- new net: DL8.2 (A), UAND_10.13, UFLIP_20.9 (Q)
- new net: C31.1, R65.2, R81.2, UFLIP_8.3 (C)
- new net: R164.1, SW62.2
- new net: C30.1, R64.2, R80.2, UFLIP_7.11 (C)
- new net: UFLIP_7.12 (D), UFLIP_7.8 (~Q)
- new net: DL32.2 (A), UAND_4.5, UFLIP_7.9 (Q)
- new net: D40.1 (K), UAND_14.11
- new net: DL44.2 (A), UAND_14.13, UFLIP_28.9 (Q)
- new net: R163.1, SW61.2
- new net: R29.1, SW12.2
- new net: C12.1, R29.2, R37.2, UFLIP_18.11 (C)
- new net: UFLIP_31.2 (D), UFLIP_31.6 (~Q)
- new net: C53.1, R155.2, R171.2, UFLIP_31.3 (C)
- new net: DL59.2 (A), UAND_16.2, UFLIP_31.5 (Q)
- new net: C45.1, R113.2, R129.2, UFLIP_11.3 (C)
- new net: D48.1 (K), UAND_6.11
- new net: C58.1, R160.2, R176.2, UFLIP_13.11 (C)
- new net: UFLIP_13.12 (D), UFLIP_13.8 (~Q)
- new net: DL64.2 (A), UAND_7.5, UFLIP_13.9 (Q)
- new net: DL62.1 (K), R190.1
- new net: D20.1 (K), UAND_11.11
- new net: D17.2 (A), D18.2 (A), D19.2 (A), D20.2 (A), D21.2 (A), D22.2 (A), D23.2 (A), D24.2 (A), UAND_18.4
- new net: DL57.1 (K), R185.1
- new net: DL57.2 (A), UAND_15.10, UFLIP_30.5 (Q)
- new net: C36.1, R104.2, R120.2, UFLIP_26.11 (C)
- new net: UFLIP_26.12 (D), UFLIP_26.8 (~Q)
- new net: DL40.2 (A), UAND_13.13, UFLIP_26.9 (Q)
- new net: D37.1 (K), UAND_14.3
- new net: DL20.1 (K), R84.1
- new net: C62.1, R164.2, R180.2, UFLIP_15.11 (C)
- new net: C38.1, R106.2, R122.2, UFLIP_27.11 (C)
- new net: D47.1 (K), UAND_6.8
- new net: D56.1 (K), UAND_16.11
- new net: DL62.2 (A), UAND_16.13, UFLIP_32.9 (Q)
- new net: DL19.1 (K), R83.1
- new net: DL19.2 (A), UAND_11.2, UFLIP_21.5 (Q)
- new net: D50.1 (K), UAND_15.6
- new net: D49.2 (A), D50.2 (A), D51.2 (A), D52.2 (A), D53.2 (A), D54.2 (A), D55.2 (A), D56.2 (A), UAND_18.12
- new net: DL66.1 (K), R194.1
- new net: UFLIP_25.2 (D), UFLIP_25.6 (~Q)
- new net: C33.1, R101.2, R117.2, UFLIP_25.3 (C)
- new net: DL37.2 (A), UAND_13.2, UFLIP_25.5 (Q)
- new net: DL37.1 (K), R133.1
- new net: D43.1 (K), UAND_5.8
- new net: R111.1, SW43.2
- new net: D42.1 (K), UAND_5.6
- new net: C37.1, R105.2, R121.2, UFLIP_27.3 (C)
- new net: UFLIP_18.12 (D), UFLIP_18.8 (~Q)
- new net: DL4.2 (A), UAND_9.13, UFLIP_18.9 (Q)
- new net: R155.1, SW53.2
- new net: D30.1 (K), UAND_4.6
- new net: R59.1, SW25.2
- new net: C24.1, R58.2, R74.2, UFLIP_24.11 (C)
- new net: DL20.2 (A), UAND_11.5, UFLIP_21.9 (Q)
- new net: D61.1 (K), UAND_8.3
- new net: UFLIP_15.12 (D), UFLIP_15.8 (~Q)
- new net: DL68.2 (A), UAND_8.5, UFLIP_15.9 (Q)
- new net: R26.1, SW9.2
- new net: R31.1, SW14.2
- new net: D62.1 (K), UAND_8.6
- new net: DL34.1 (K), R98.1
- new net: D46.1 (K), UAND_6.6
- new net: R53.1, SW19.2
- new net: DL43.2 (A), UAND_14.10, UFLIP_28.5 (Q)
- new net: D39.1 (K), UAND_14.8
- new net: DL53.2 (A), JOUT5.T, UAND_18.8
- new net: C29.1, R63.2, R79.2, UFLIP_7.3 (C)
- new net: C10.1, R27.2, R35.2, UFLIP_17.11 (C)
- new net: R115.1, SW47.2
- new net: DL23.2 (A), UAND_12.2, UFLIP_23.5 (Q)
- new net: D21.1 (K), UAND_12.3
- new net: R64.1, SW30.2
- new net: R165.1, SW63.2
- new net: D11.1 (K), UAND_9.8
- new net: D10.2 (A), D11.2 (A), D12.2 (A), D13.2 (A), D14.2 (A), D15.2 (A), D16.2 (A), D9.2 (A), UAND_18.1
- new net: D27.1 (K), UAND_3.8
- new net: DL36.1 (K), R100.1
- new net: R107.1, SW39.2
- new net: C54.1, R156.2, R172.2, UFLIP_31.11 (C)
- new net: C60.1, R162.2, R178.2, UFLIP_14.11 (C)
- new net: C20.1, R54.2, R70.2, UFLIP_22.11 (C)
- new net: R28.1, SW11.2
- new net: C11.1, R28.2, R36.2, UFLIP_18.3 (C)
- new net: DL31.1 (K), R95.1
- new net: R102.1, SW34.2
- new net: C34.1, R102.2, R118.2, UFLIP_25.11 (C)
- new net: C46.1, R114.2, R130.2, UFLIP_11.11 (C)
- new net: DL41.1 (K), R137.1
- new net: DL23.1 (K), R87.1
- new net: R109.1, SW41.2
- new net: R61.1, SW27.2
- new net: C17.1, R51.2, R67.2, UFLIP_21.3 (C)
- new net: DL51.1 (K), R147.1
- new net: DL51.2 (A), UAND_6.10, UFLIP_12.5 (Q)
- new net: R65.1, SW31.2
- new net: R112.1, SW44.2
- new net: D14.1 (K), UAND_10.6
- new net: DL35.2 (A), JOUT3.T, UAND_18.6
- new net: UFLIP_27.12 (D), UFLIP_27.8 (~Q)
- new net: D18.1 (K), UAND_11.6
- new net: R159.1, SW57.2
- new net: DL65.1 (K), R193.1
- new net: DL33.1 (K), R97.1
- new net: DL33.2 (A), UAND_4.10, UFLIP_8.5 (Q)
- new net: D24.1 (K), UAND_12.11
- new net: DL26.2 (A), UAND_12.13, UFLIP_24.9 (Q)
- new net: R30.1, SW13.2
- new net: R105.1, SW37.2
- new net: DL59.1 (K), R187.1
- new net: R153.1, SW51.2
- new net: DL3.1 (K), R44.1
- new net: DL3.2 (A), UAND_9.10, UFLIP_18.5 (Q)
- new net: UFLIP_10.12 (D), UFLIP_10.8 (~Q)
- new net: DL63.1 (K), R191.1
- new net: DL63.2 (A), UAND_7.2, UFLIP_13.5 (Q)
- new net: UFLIP_13.2 (D), UFLIP_13.6 (~Q)
- new net: C57.1, R159.2, R175.2, UFLIP_13.3 (C)
- new net: R152.1, SW50.2
- new net: DL67.1 (K), R195.1
- new net: UFLIP_14.12 (D), UFLIP_14.8 (~Q)
- new net: D17.1 (K), UAND_11.3
- new net: UFLIP_5.2 (D), UFLIP_5.6 (~Q)
- new net: DL27.2 (A), UAND_3.2, UFLIP_5.5 (Q)
- new net: DL4.1 (K), R45.1
- new net: DL61.1 (K), R189.1
- new net: D51.1 (K), UAND_15.8
- new net: DL54.1 (K), R150.1
- new net: R116.1, SW48.2
- new net: DL38.1 (K), R134.1
- new net: DL48.1 (K), R144.1
- new net: UFLIP_29.12 (D), UFLIP_29.8 (~Q)
- new net: DL56.2 (A), UAND_15.5, UFLIP_29.9 (Q)
- new net: C47.1, R115.2, R131.2, UFLIP_12.3 (C)
- new net: C43.1, R111.2, R127.2, UFLIP_10.3 (C)
- new net: C39.1, R107.2, R123.2, UFLIP_28.3 (C)
- new net: R166.1, SW64.2
- new net: C64.1, R166.2, R182.2, UFLIP_16.11 (C)
- new net: DL35.1 (K), R99.1
- new net: D55.1 (K), UAND_16.8
- new net: UFLIP_7.2 (D), UFLIP_7.6 (~Q)
- new net: DL31.2 (A), UAND_4.2, UFLIP_7.5 (Q)
- new net: R104.1, SW36.2
- new net: DL1.2 (A), UAND_9.2, UFLIP_17.5 (Q)
- new net: D9.1 (K), UAND_9.3
- new net: UFLIP_8.2 (D), UFLIP_8.6 (~Q)
- new net: DL24.1 (K), R88.1
- new net: UFLIP_22.2 (D), UFLIP_22.6 (~Q)
- new net: C19.1, R53.2, R69.2, UFLIP_22.3 (C)
- new net: DL21.2 (A), UAND_11.10, UFLIP_22.5 (Q)
- new net: UFLIP_29.2 (D), UFLIP_29.6 (~Q)
- new net: C49.1, R151.2, R167.2, UFLIP_29.3 (C)
- new net: DL55.2 (A), UAND_15.2, UFLIP_29.5 (Q)
- new net: R62.1, SW28.2
- new net: D16.1 (K), UAND_10.11
- new net: R63.1, SW29.2
- new net: R33.1, SW16.2
- new net: R51.1, SW17.2
- new net: DL27.1 (K), R91.1
- new net: DL45.2 (A), UAND_5.2, UFLIP_9.5 (Q)
- new net: UFLIP_24.12 (D), UFLIP_24.8 (~Q)
- new net: C63.1, R165.2, R181.2, UFLIP_16.3 (C)
- new net: UFLIP_9.2 (D), UFLIP_9.6 (~Q)
- new net: C41.1, R109.2, R125.2, UFLIP_9.3 (C)
- new net: C16.1, R33.2, R41.2, UFLIP_20.11 (C)
- new net: DL18.2 (A), JOUT2.T, UAND_18.3
- new net: DL38.2 (A), UAND_13.5, UFLIP_25.9 (Q)
- new net: D34.1 (K), UAND_13.6
- new net: C61.1, R163.2, R179.2, UFLIP_15.3 (C)
- new net: UFLIP_16.12 (D), UFLIP_16.8 (~Q)
- new net: UFLIP_15.2 (D), UFLIP_15.6 (~Q)
- new net: DL67.2 (A), UAND_8.2, UFLIP_15.5 (Q)
- new net: D49.1 (K), UAND_15.3
- new net: DL7.1 (K), R48.1
- new net: DL7.2 (A), UAND_10.10, UFLIP_20.5 (Q)
- new net: C51.1, R153.2, R169.2, UFLIP_30.3 (C)
- new net: R157.1, SW55.2
- new net: DL6.1 (K), R47.1
- new net: UFLIP_31.12 (D), UFLIP_31.8 (~Q)
- new net: DL60.2 (A), UAND_16.5, UFLIP_31.9 (Q)
- new net: C23.1, R57.2, R73.2, UFLIP_24.3 (C)
- new net: D54.1 (K), UAND_16.6
- new net: DL72.1 (K), R200.1
- new net: DL26.1 (K), R90.1
- new net: DL52.2 (A), UAND_6.13, UFLIP_12.9 (Q)
- new net: D23.1 (K), UAND_12.8
- new net: R160.1, SW58.2
- new net: DL60.1 (K), R188.1
- new net: R57.1, SW23.2
- new net: D22.1 (K), UAND_12.6
- new net: C56.1, R158.2, R174.2, UFLIP_32.11 (C)
- new net: UFLIP_32.12 (D), UFLIP_32.8 (~Q)
- new net: C48.1, R116.2, R132.2, UFLIP_12.11 (C)
- new net: R162.1, SW60.2
- new net: DL32.1 (K), R96.1
- new net: DL5.1 (K), R46.1
- new net: UFLIP_14.2 (D), UFLIP_14.6 (~Q)
- new net: C59.1, R161.2, R177.2, UFLIP_14.3 (C)
- new net: R161.1, SW59.2
- new net: DL50.1 (K), R146.1
- new net: DL70.1 (K), R198.1
- new net: C13.1, R30.2, R38.2, UFLIP_19.3 (C)
- new net: DL64.1 (K), R192.1
- new net: DL49.1 (K), R145.1
- new net: DL49.2 (A), UAND_6.2, UFLIP_11.5 (Q)
- new net: DL71.1 (K), R199.1
- new net: DL71.2 (A), JOUT7.T, UAND_18.11
- new net: DL43.1 (K), R139.1
- new net: DL30.1 (K), R94.1
- new net: DL30.2 (A), UAND_3.13, UFLIP_6.9 (Q)
- new net: DL58.1 (K), R186.1
- new net: UFLIP_10.2 (D), UFLIP_10.6 (~Q)
- new net: DL5.2 (A), UAND_10.2, UFLIP_19.5 (Q)
- new net: D13.1 (K), UAND_10.3
- new net: C26.1, R60.2, R76.2, UFLIP_5.11 (C)
- new net: R54.1, SW20.2
- new net: R156.1, SW54.2
- new net: R151.1, SW49.2
- new net: DL22.2 (A), UAND_11.13, UFLIP_22.9 (Q)
- new net: DL28.1 (K), R92.1
- new net: DL28.2 (A), UAND_3.5, UFLIP_5.9 (Q)
- new net: UFLIP_25.12 (D), UFLIP_25.8 (~Q)
- new net: DL50.2 (A), UAND_6.5, UFLIP_11.9 (Q)
- new net: DL25.1 (K), R89.1
- new net: DL61.2 (A), UAND_16.10, UFLIP_32.5 (Q)
- new net: UFLIP_16.2 (D), UFLIP_16.6 (~Q)
- new net: UFLIP_12.2 (D), UFLIP_12.6 (~Q)
- new net: R55.1, SW21.2
- new net: C21.1, R55.2, R71.2, UFLIP_23.3 (C)
- new net: D25.1 (K), UAND_3.3
- new net: DL22.1 (K), R86.1
- new net: DL1.1 (K), R42.1
- new net: D12.1 (K), UAND_9.11
- new net: D41.1 (K), UAND_5.3
- new net: D52.1 (K), UAND_15.11
- new net: R60.1, SW26.2
- new net: D57.1 (K), UAND_7.3
- new net: D26.1 (K), UAND_3.6
- new net: R58.1, SW24.2
- new net: UFLIP_28.2 (D), UFLIP_28.6 (~Q)
- new net: D28.1 (K), UAND_3.11
- new net: DL25.2 (A), UAND_12.10, UFLIP_24.5 (Q)
- new net: C35.1, R103.2, R119.2, UFLIP_26.3 (C)
- new net: D31.1 (K), UAND_4.8
- new net: D53.1 (K), UAND_16.3
- new net: D15.1 (K), UAND_10.8
- new net: D32.1 (K), UAND_4.11
- new net: DL21.1 (K), R85.1
- new net: R32.1, SW15.2
- new net: C15.1, R32.2, R40.2, UFLIP_20.3 (C)
- new net: DL41.2 (A), UAND_14.2, UFLIP_27.5 (Q)
- new net: D36.1 (K), UAND_13.11
- new net: DL56.1 (K), R184.1
- new net: D35.1 (K), UAND_13.8
- new net: UFLIP_32.2 (D), UFLIP_32.6 (~Q)
- new net: C55.1, R157.2, R173.2, UFLIP_32.3 (C)
- new net: DL40.1 (K), R136.1
- new net: R56.1, SW22.2
- new net: UFLIP_19.2 (D), UFLIP_19.6 (~Q)
- new net: UFLIP_20.12 (D), UFLIP_20.8 (~Q)
- new net: UFLIP_17.12 (D), UFLIP_17.8 (~Q)
- new net: UFLIP_17.2 (D), UFLIP_17.6 (~Q)
- new net: DL29.1 (K), R93.1
- new net: UFLIP_9.12 (D), UFLIP_9.8 (~Q)
- new net: UFLIP_27.2 (D), UFLIP_27.6 (~Q)
- new net: R101.1, SW33.2
- new net: UFLIP_23.2 (D), UFLIP_23.6 (~Q)
- new net: C40.1, R108.2, R124.2, UFLIP_28.11 (C)
- new net: DL44.1 (K), R140.1
- new net: D19.1 (K), UAND_11.8
- new net: UFLIP_6.12 (D), UFLIP_6.8 (~Q)
- new net: D33.1 (K), UAND_13.3
- new net: UFLIP_21.2 (D), UFLIP_21.6 (~Q)
- new net: DL29.2 (A), UAND_3.10, UFLIP_6.5 (Q)
- new net: UFLIP_18.2 (D), UFLIP_18.6 (~Q)
- new net: UFLIP_5.12 (D), UFLIP_5.8 (~Q)
- new net: D45.1 (K), UAND_6.3
- new net: R114.1, SW46.2
- new net: D10.1 (K), UAND_9.6
- new net: UFLIP_11.12 (D), UFLIP_11.8 (~Q)
- new net: UFLIP_24.2 (D), UFLIP_24.6 (~Q)
- new net: D29.1 (K), UAND_4.3
- new net: UFLIP_12.12 (D), UFLIP_12.8 (~Q)
- new net: UFLIP_6.2 (D), UFLIP_6.6 (~Q)
- new net: UFLIP_21.12 (D), UFLIP_21.8 (~Q)
- new net: UFLIP_30.2 (D), UFLIP_30.6 (~Q)
- new net: UFLIP_28.12 (D), UFLIP_28.8 (~Q)
- new net: R154.1, SW52.2
- new net: UFLIP_26.2 (D), UFLIP_26.6 (~Q)
- new net: UFLIP_11.2 (D), UFLIP_11.6 (~Q)
- new net: UFLIP_22.12 (D), UFLIP_22.8 (~Q)
- new net: R158.1, SW56.2
- new net: UFLIP_20.2 (D), UFLIP_20.6 (~Q)
Other:
- moved on the sheet: J1, UAND_17B, UAND_17C, UAND_17D, UFLIP_1C, UFLIP_2C, UFLIP_3C, UFLIP_4C
